Commit message: Update compoenent positions in urdf.

File: dagny_model/dagny.urdf (robot description, URDF)
Before this commit: robot dagny, 6 links, 5 joints
Joints:
- joint fl_wheel_joint: origin xyz=0.34 0.12 0 rpy=1.57 0 0 -> xyz=0.335 0.12 0.055 rpy=1.57 0 0
- joint fr_wheel_joint: origin xyz=0.34 -0.12 0 rpy=1.57 0 0 -> xyz=0.335 -0.12 0.055 rpy=1.57 0 0
- joint rl_wheel_joint: origin xyz=0 0.12 0 rpy=1.57 0 0 -> xyz=0 0.12 0.055 rpy=1.57 0 0
- joint rr_wheel_joint: origin xyz=0 -0.12 0 rpy=1.57 0 0 -> xyz=0 -0.12 0.055 rpy=1.57 0 0

Commit message: Add sonars to URDF.

File: dagny_model/dagny.urdf (robot description, URDF)
Before this commit: robot dagny, 6 links, 5 joints
Links:
- added link sonar_1
- added link sonar_2
- added link sonar_3
- added link sonar_4
- added link sonar_5
Joints:
- added joint sonar_1_joint: type fixed, parent base_link, child sonar_1, origin xyz=0.38 -0.06 0.10 rpy=0 0 -0.7854
- added joint sonar_2_joint: type fixed, parent base_link, child sonar_2, origin xyz=0.40 0 0.10 rpy=0 0 0
- added joint sonar_3_joint: type fixed, parent base_link, child sonar_3, origin xyz=0.38 0.06 0.10 rpy=0 0 0.7854
- added joint sonar_4_joint: type fixed, parent base_link, child sonar_4, origin xyz=-0.12 0.05 0.10 rpy=0 0 2.74
- added joint sonar_5_joint: type fixed, parent base_link, child sonar_5, origin xyz=-0.12 -0.05 0.10 rpy=0 0 -2.74
